Commit message: demo_pretrain_best_last

File: aliengo_description/urdf/aliengo.urdf (robot description, URDF)
Before this commit: robot aliengo, 19 links, 18 joints
Links:
- removed link base
Joints:
- removed joint floating_base
- joint FL_hip_joint: limit lower=-1.2217304764 upper=1.2217304764 effort=44.4 velocity=40 -> lower=-0.2217304764 upper=0.2217304764 effort=44.4 velocity=40
- joint FL_thigh_joint: limit lower=-1.2217304764 upper=1.2217304764 effort=44.4 velocity=40 -> lower=0.2217304764 upper=1.2217304764 effort=44.4 velocity=40
- joint FR_hip_joint: limit lower=-1.2217304764 upper=1.2217304764 effort=44.4 velocity=40 -> lower=-0.2217304764 upper=0.2217304764 effort=44.4 velocity=40
- joint FR_thigh_joint: limit lower=-1.2217304764 upper=1.2217304764 effort=44.4 velocity=40 -> lower=0.2217304764 upper=1.2217304764 effort=44.4 velocity=40
- joint RL_hip_joint: limit lower=-1.2217304764 upper=1.2217304764 effort=44.4 velocity=40 -> lower=0.2217304764 upper=0.2217304764 effort=44.4 velocity=40
- joint RL_thigh_joint: limit lower=-1.2217304764 upper=1.2217304764 effort=44.4 velocity=40 -> lower=0.2217304764 upper=1.2217304764 effort=44.4 velocity=40
- joint RR_hip_joint: limit lower=-1.2217304764 upper=1.2217304764 effort=44.4 velocity=40 -> lower=-0.2217304764 upper=0.2217304764 effort=44.4 velocity=40
- joint RR_thigh_joint: limit lower=-1.2217304764 upper=1.2217304764 effort=44.4 velocity=40 -> lower=0.2217304764 upper=1.2217304764 effort=44.4 velocity=40
